Commit message: Change names in robot model to be more descriptive and follow conventions

File: metralabs_ros/models/scitos_haw_schunk.urdf (robot description, URDF)
Before this commit: robot scitos_haw_schunk, 16 links, 15 joints
Links:
- removed link CameraMount
- removed link ConnBase
- removed link ConnLong1
- removed link ConnLong2
- removed link DH1
- removed link DH2
- removed link DH3
- removed link DH4
- removed link DH5
- removed link DH6
- removed link GFneg
- removed link GFpos
- removed link Gripper
- removed link Kinect
- added link arm_base_connector; visual cylinder length=0.060 radius=0.080
- added link arm_base_link
- added link arm_link_1; collision cylinder length=0.118 radius=0.0833333333333; visual cylinder length=0.13 radius=0.05
- added link arm_link_2; collision cylinder length=0.118 radius=0.0833333333333; visual cylinder length=0.13 radius=0.05
- added link arm_link_2_connector; collision box size=0.51 0.110 0.08; visual box size=0.47 0.105 0.038
- added link arm_link_3; collision cylinder length=0.118 radius=0.0833333333333; visual cylinder length=0.13 radius=0.05
- added link arm_link_3_connector; collision box size=0.41 0.110 0.08; visual box size=0.37 0.105 0.038
- added link arm_link_4; collision cylinder length=0.118 radius=0.0666666666667; visual cylinder length=0.104 radius=0.04
- added link arm_link_5; collision cylinder length=0.118 radius=0.05; visual cylinder length=0.078 radius=0.03
- added link camera_mount; collision box size=0.090 0.070 0.030; visual box size=0.073 0.051 0.025
- added link gripper; collision box size=0.185 0.100 0.132; visual box size=0.090 0.080 0.112
- added link gripper_finger_neg; visual box size=0.070 0.030 0.020
- added link gripper_finger_pos; visual box size=0.070 0.030 0.020
- added link kinect; collision box size=0.08 0.30 0.06; visual box size=0.06 0.28 0.04
Joints:
- removed joint CameraMount_Kinect
- removed joint DH1_ConnBase
- removed joint DH3_ConnLong1
- removed joint DH4_ConnLong2
- removed joint DH_1_2
- removed joint DH_2_3
- removed joint DH_3_4
- removed joint DH_4_5
- removed joint DH_5_6
- removed joint DH_6_GR
- removed joint DH_B_1
- removed joint GR_Fneg
- removed joint GR_Fpos
- removed joint Gripper_CameraMount
- added joint arm_base_fixing: type fixed, parent base_link, child arm_base_link, origin xyz=-0.075 0 0.583 rpy=0 0 0
- added joint arm_base_link_arm_base_connector: type fixed, parent arm_base_link, child arm_base_connector, origin xyz=0 0 0 rpy=0 0 0
- added joint arm_joint_1: type revolute, parent arm_base_link, child arm_link_1, origin xyz=0 0 0.120 rpy=0 0 0, axis 0 0 -1, limit lower=-3.141593 upper=3.141593 effort=2 velocity=0.437
- added joint arm_joint_2: type revolute, parent arm_link_1, child arm_link_2, origin xyz=0 0 0.148 rpy=1.57079632679 -1.57079632679 3.14159265359, axis 0 0 -1, limit lower=-2.024580 upper=2.024580 effort=2 velocity=0.438
- added joint arm_joint_3: type revolute, parent arm_link_2, child arm_link_3, origin xyz=0.400 0 0 rpy=3.14159265359 0 0, axis 0 0 -1, limit lower=-2.740166 upper=2.740166 effort=2 velocity=0.436
- added joint arm_joint_4: type revolute, parent arm_link_3, child arm_link_4, origin xyz=0.300 0 0 rpy=3.14159265359 0 0, axis 0 0 -1, limit lower=-2.373644 upper=2.286380 effort=2 velocity=0.486
- added joint arm_joint_5: type revolute, parent arm_link_4, child arm_link_5, origin xyz=0.121 0 0 rpy=0 1.57079632679 0, axis 0 0 -1, limit lower=-3.143321 upper=3.143321 effort=2 velocity=0.872
- added joint arm_link_2_arm_link_2_connector: type fixed, parent arm_link_2, child arm_link_2_connector, origin xyz=0 0 0 rpy=0 0 0
- added joint arm_link_3_arm_link_3_connector: type fixed, parent arm_link_3, child arm_link_3_connector, origin xyz=0 0 0 rpy=0 0 0
- added joint camera_mount_kinect: type fixed, parent camera_mount, child kinect, origin xyz=-0.015 0 0.04 rpy=0 0 0
- added joint gripper_camera_mount: type fixed, parent gripper, child camera_mount, origin xyz=-0.011 -0.055 0 rpy=1.57079632679 0 0
- added joint gripper_fixing: type fixed, parent arm_link_5, child gripper, origin xyz=0 0 0.130 rpy=0 -1.57079632679 0
- added joint gripper_joint_neg: type prismatic, parent gripper, child gripper_finger_neg, origin xyz=0.047 0 0 rpy=0 0 0, axis 0 0 1, limit lower=-0.000250 upper=0.068111 effort=2 velocity=0.08, mimic joint=gripper_joint_pos multiplier=0.5 offset=0
- added joint gripper_joint_pos: type prismatic, parent gripper_finger_neg, child gripper_finger_pos, origin xyz=0 0 0 rpy=3.14159265359 0 0, axis 0 0 1, limit lower=-0.000250 upper=0.068111 effort=2 velocity=0.08

File: metralabs_ros/models/xacro/scitos_haw_schunk.xacro (robot description, xacro)
@@ -6,19 +6,19 @@
 <!-- Joints macros -->
 <xacro:include filename="$(find metralabs_ros)/models/xacro/scitos_haw_schunk_joints.xacro" />
-<xacro:DH  name="DH1"/><!-- base of arm -->
-<xacro:PRL name="DH2" type="100"/><!-- ~center of base swivel joint ID20 -->
-<xacro:PRL name="DH3" type="100"/><!-- center of first pitch joint ID21 -->
-<xacro:PRL name="DH4" type="100"/><!-- center of second pitch joint ID22 -->
-<xacro:PRL name="DH5" type="80"/><!-- center of third pitch joint ID23 -->
-<xacro:PRL name="DH6" type="60"/><!-- center of hand roll joint ID24 -->
-<xacro:Connector name="ConnBase" >
+<xacro:DH  name="arm_base_link"/><!-- base of arm -->
+<xacro:PRL name="arm_link_1" type="100"/><!-- ~center of base swivel joint ID20 -->
+<xacro:PRL name="arm_link_2" type="100"/><!-- center of first pitch joint ID21 -->
+<xacro:PRL name="arm_link_3" type="100"/><!-- center of second pitch joint ID22 -->
+<xacro:PRL name="arm_link_4" type="80"/><!-- center of third pitch joint ID23 -->
+<xacro:PRL name="arm_link_5" type="60"/><!-- center of hand roll joint ID24 -->
+<xacro:Connector name="arm_base_connector" >
     <cylinder radius="0.080" length="0.060" /> <!--values ok-->
 </xacro:Connector>
-<xacro:connect parent="DH1" child="ConnBase"/>
-<xacro:Connector_long name="ConnLong1" length="400"/>
-<xacro:Connector_long name="ConnLong2" length="300"/>
-<xacro:connect parent="DH3" child="ConnLong1"/>
-<xacro:connect parent="DH4" child="ConnLong2"/>
-<link name="Gripper">
+<xacro:connect parent="arm_base_link" child="arm_base_connector"/>
+<xacro:Connector_long name="arm_link_2_connector" length="400"/>
+<xacro:Connector_long name="arm_link_3_connector" length="300"/>
+<xacro:connect parent="arm_link_2" child="arm_link_2_connector"/>
+<xacro:connect parent="arm_link_3" child="arm_link_3_connector"/>
+<link name="gripper">
   <visual>
     <origin xyz="0 0 0" rpy="0 0 0" />
@@ -35,9 +35,9 @@
   </collision>
 </link>
-<xacro:GripperFinger name="GFpos" reflect="1"/>
-<!--<xacro:connect parent="Gripper" child="GFpos"/>-->
-<xacro:GripperFinger name="GFneg" reflect="-1"/>
-<!--<xacro:connect parent="Gripper" child="GFneg"/>-->
-<link name="CameraMount">
+<xacro:GripperFinger name="gripper_finger_pos" reflect="1"/>
+<!--<xacro:connect parent="gripper" child="gripper_finger_pos"/>-->
+<xacro:GripperFinger name="gripper_finger_neg" reflect="-1"/>
+<!--<xacro:connect parent="gripper" child="gripper_finger_neg"/>-->
+<link name="camera_mount">
   <visual>
     <origin xyz="-0.0085 0 -0.003210" rpy="0 0 0" />
@@ -53,6 +53,6 @@
   </collision>
 </link>
-<xacro:connect_xyz_rpy parent="Gripper" child="CameraMount" xyz="-0.011 -0.055 0" rpy="${0.25*tau} 0 0"/><!-- Werte berechnet -->
-<link name="Kinect">
+<xacro:connect_xyz_rpy parent="gripper" child="camera_mount" xyz="-0.011 -0.055 0" rpy="${0.25*tau} 0 0"/><!-- Werte berechnet -->
+<link name="kinect">
   <visual>
     <geometry>
@@ -67,4 +67,4 @@
   </collision>
 </link>
-<xacro:connect_xyz parent="CameraMount" child="Kinect" xyz="-0.015 0 0.04"/><!-- Werte auf cm vermessen -->
+<xacro:connect_xyz parent="camera_mount" child="kinect" xyz="-0.015 0 0.04"/><!-- Werte auf cm vermessen -->
 </robot>

File: metralabs_ros/models/xacro/scitos_haw_schunk_joints.xacro (robot description, xacro)
@@ -1,109 +1,109 @@
 <robot xmlns:xacro="http://ros.org/wiki/xacro">
- <joint name="DH_B_1" type="fixed">
+ <joint name="arm_base_fixing" type="fixed">
     <origin xyz="${schunk_base_offset_center} 0 ${scitos_height}" rpy="0 0 0"/>
     <parent link="base_link"/>
-    <child link="DH1"/>
+    <child link="arm_base_link"/>
  </joint>
- <joint name="DH_1_2" type="revolute">
+ <joint name="arm_joint_1" type="revolute">
 	<!-- ~center of base swivel joint ID20 -->
     <!-- the ~center means: both z of this and below added must equal 0.268 to match reality -->
     <origin xyz="0 0 0.120" rpy="0 0 0"/>
-    <parent link="DH1"/>
-    <child link="DH2"/>
+    <parent link="arm_base_link"/>
+    <child link="arm_link_1"/>
     <axis xyz="0 0 -1" />
     <limit lower="-3.141593" upper="3.141593" effort="2" velocity="0.437" />
  </joint>
- <joint name="DH_2_3" type="revolute">
+ <joint name="arm_joint_2" type="revolute">
 	<!-- center of first pitch joint ID21 -->
     <origin xyz="0 0 0.148" rpy="${0.25*tau} ${-0.25*tau} ${0.5*tau}"/>
-    <parent link="DH2"/>
-    <child link="DH3"/>
+    <parent link="arm_link_1"/>
+    <child link="arm_link_2"/>
     <axis xyz="0 0 -1" />
     <limit lower="-2.024580" upper="2.024580" effort="2" velocity="0.438" />
  </joint>
- <joint name="DH_3_4" type="revolute">
+ <joint name="arm_joint_3" type="revolute">
     <!-- center of second pitch joint ID22 -->
     <origin xyz="0.400 0 0" rpy="${0.5*tau} 0 0"/>
-    <parent link="DH3"/>
-    <child link="DH4"/>
+    <parent link="arm_link_2"/>
+    <child link="arm_link_3"/>
     <axis xyz="0 0 -1" />
     <limit lower="-2.740166" upper="2.740166" effort="2" velocity="0.436" />
  </joint>
- <joint name="DH_4_5" type="revolute">
+ <joint name="arm_joint_4" type="revolute">
 	<!-- center of third pitch joint ID23 -->
     <origin xyz="0.300 0 0" rpy="${0.5*tau} 0 0"/>
-    <parent link="DH4"/>
-    <child link="DH5"/>
+    <parent link="arm_link_3"/>
+    <child link="arm_link_4"/>
     <axis xyz="0 0 -1" />
     <limit lower="-2.373644" upper="2.286380" effort="2" velocity="0.486" />
  </joint>
- <joint name="DH_5_6" type="revolute">
+ <joint name="arm_joint_5" type="revolute">
 	<!-- center of hand roll joint ID24 -->
     <origin xyz="0.121 0 0" rpy="0 ${0.25*tau} 0"/>
-    <parent link="DH5"/>
-    <child link="DH6"/>
+    <parent link="arm_link_4"/>
+    <child link="arm_link_5"/>
     <axis xyz="0 0 -1" />
     <limit lower="-3.143321" upper="3.143321" effort="2" velocity="0.872" />
  </joint>
- <joint name="DH_6_GR" type="fixed">
+ <joint name="gripper_fixing" type="fixed">
     <origin xyz="0 0 0.130" rpy="0 ${-0.25*tau} 0"/>
-    <parent link="DH6"/>
-    <child link="Gripper"/>
+    <parent link="arm_link_5"/>
+    <child link="gripper"/>
  </joint>
- <joint name="GR_Fpos" type="prismatic">
+ <joint name="gripper_joint_pos" type="prismatic">
     <origin xyz="0 0 0" rpy="${0.5*tau} 0 0"/>
-    <parent link="GFneg"/>
-    <child link="GFpos"/>
+    <parent link="gripper_finger_neg"/>
+    <child link="gripper_finger_pos"/>
     <axis xyz="0 0 1" />
     <limit lower="-0.000250" upper="0.068111" effort="2" velocity="0.08" />
  </joint>
- <joint name="GR_Fneg" type="prismatic">
+ <joint name="gripper_joint_neg" type="prismatic">
     <origin xyz="0.047 0 0" rpy="0 0 0"/>
-    <parent link="Gripper"/>
-    <child link="GFneg"/>
+    <parent link="gripper"/>
+    <child link="gripper_finger_neg"/>
     <axis xyz="0 0 1" />
     <limit lower="-0.000250" upper="0.068111" effort="2" velocity="0.08" />
-    <mimic joint="GR_Fpos" multiplier="0.5" offset="0"/>
+    <mimic joint="gripper_joint_pos" multiplier="0.5" offset="0"/>
  </joint>
 <!-- Backup: rechtsdrehende Gelenke
- <joint name="DH_B_1" type="fixed">
+ <joint name="arm_base_fixing" type="fixed">
     <origin xyz="0 0 0.700" rpy="0 0 0"/>
     <parent link="ScitosBase"/>
-    <child link="DH1"/>
+    <child link="arm_base_link"/>
     <axis xyz="0 0 1" />
     <limit lower="-3.0543" upper="3.0543" effort="2" velocity="${max_vel}" />
  </joint>
- <joint name="DH_1_2" type="revolute">
+ <joint name="arm_joint_1" type="revolute">
     <origin xyz="0 0 0.060" rpy="0 0 ${0.5*tau}"/>
-    <parent link="DH1"/>
-    <child link="DH2"/>
+    <parent link="arm_base_link"/>
+    <child link="arm_link_1"/>
     <axis xyz="0 0 1" />
     <limit lower="-3.0543" upper="3.0543" effort="2" velocity="${max_vel}" />
  </joint>
- <joint name="DH_2_3" type="revolute">
+ <joint name="arm_joint_2" type="revolute">
     <origin xyz="0 0 0.208" rpy="${0.25*tau} ${-0.25*tau} ${0.5*tau}"/>
-    <parent link="DH2"/>
-    <child link="DH3"/>
+    <parent link="arm_link_1"/>
+    <child link="arm_link_2"/>
     <axis xyz="0 0 1" />
     <limit lower="-3.0543" upper="3.0543" effort="2" velocity="${max_vel}" />
  </joint>
- <joint name="DH_3_4" type="revolute">
+ <joint name="arm_joint_3" type="revolute">
     <origin xyz="0.400 0 0" rpy="${0.5*tau} 0 0"/>
-    <parent link="DH3"/>
-    <child link="DH4"/>
+    <parent link="arm_link_2"/>
+    <child link="arm_link_3"/>
     <axis xyz="0 0 1" />
     <limit lower="-3.0543" upper="3.0543" effort="2" velocity="${max_vel}" />
  </joint>
- <joint name="DH_4_5" type="revolute">
+ <joint name="arm_joint_4" type="revolute">
     <origin xyz="0.300 0 0" rpy="${0.5*tau} 0 0"/>
-    <parent link="DH4"/>
-    <child link="DH5"/>
+    <parent link="arm_link_3"/>
+    <child link="arm_link_4"/>
     <axis xyz="0 0 1" />
     <limit lower="-3.0543" upper="3.0543" effort="2" velocity="${max_vel}" />
  </joint>
- <joint name="DH_5_6" type="revolute">
+ <joint name="arm_joint_5" type="revolute">
     <origin xyz="0.200 0 0" rpy="0 ${0.25*tau} 0"/>
-    <parent link="DH5"/>
-    <child link="DH6"/>
+    <parent link="arm_link_4"/>
+    <child link="arm_link_5"/>
     <axis xyz="0 0 1" />
     <limit lower="-3.0543" upper="3.0543" effort="2" velocity="${max_vel}" />
